Commit message: straight initial angles, more observations and terminations

File: exts/MARL_mav_carry_ext/MARL_mav_carry_ext/assets/data/AMR/flycrane_data/flycrane.urdf (robot description, URDF)
Before this commit: robot flycrane, 95 links, 94 joints
Joints:
- joint rope_1_sphere_joint_0_joint_x: origin xyz=0.24 0.22 0.14 rpy=-1 0 0 -> xyz=0.24 0.22 0.14 rpy=0 0 0
- joint rope_2_sphere_joint_0_joint_x: origin xyz=0.24 -0.22 0.14 rpy=1 0 0 -> xyz=0.24 -0.22 0.14 rpy=0 0 0
- joint rope_3_sphere_joint_0_joint_x: origin xyz=-0.28 0.018 0.14 rpy=0 -1 0 -> xyz=-0.28 0.018 0.14 rpy=0 0 0

Commit message: re-aligned flycrane ropes, admit torque actions and falcon angle terminations

File: exts/MARL_mav_carry_ext/MARL_mav_carry_ext/assets/data/AMR/flycrane_data/flycrane.urdf (robot description, URDF)
Before this commit: robot flycrane, 95 links, 94 joints
Joints:
- joint Falcon1/base_joint: origin xyz=0 0 0.03 rpy=0 0 0 -> xyz=0 0 0.00 rpy=0 0 0
- joint Falcon1/odometry_sensor_joint: origin xyz=0.0 0.0 0.03 rpy=0.0 0.0 0.0 -> xyz=0.0 0.0 0.0 rpy=0.0 0.0 0.0
- joint Falcon2/base_joint: origin xyz=0 0 0.03 rpy=0 0 0 -> xyz=0 0 0.0 rpy=0 0 0
- joint Falcon2/odometry_sensor_joint: origin xyz=0.0 0.0 0.03 rpy=0.0 0.0 0.0 -> xyz=0.0 0.0 0.0 rpy=0.0 0.0 0.0
- joint Falcon3/base_joint: origin xyz=0 0 0.03 rpy=0 0 0 -> xyz=0 0 0.0 rpy=0 0 0
- joint Falcon3/odometry_sensor_joint: origin xyz=0.0 0.0 0.03 rpy=0.0 0.0 0.0 -> xyz=0.0 0.0 0.0 rpy=0.0 0.0 0.0
- joint rope_1_sphere_joint_0_joint_x: origin xyz=0.24 0.22 0.14 rpy=0 0 0 -> xyz=0.27 0.22 0.14 rpy=0 0 0
- joint rope_2_sphere_joint_0_joint_x: origin xyz=0.24 -0.22 0.14 rpy=0 0 0 -> xyz=0.27 -0.22 0.14 rpy=0 0 0
- joint rope_3_sphere_joint_0_joint_x: origin xyz=-0.28 0.018 0.14 rpy=0 0 0 -> xyz=-0.27 0.0 0.14 rpy=0 0 0

Commit message: fix forward axis drone and rotor numbering

File: exts/MARL_mav_carry_ext/MARL_mav_carry_ext/assets/data/AMR/flycrane_data/flycrane.urdf (robot description, URDF)
Before this commit: robot flycrane, 95 links, 94 joints
Links:
- link Falcon1/rotor_0: geometry collision cylinder length=0.005 radius=0.127; visual mesh filename=Falcon_PropellerCW.dae scale=1.0 1.0 1.0
- link Falcon1/rotor_3: geometry collision cylinder length=0.005 radius=0.127; visual mesh filename=Falcon_PropellerCCW.dae scale=1.0 1.0 1.0
- link Falcon2/rotor_0: geometry collision cylinder length=0.005 radius=0.127; visual mesh filename=Falcon_PropellerCW.dae scale=1.0 1.0 1.0
- link Falcon2/rotor_3: geometry collision cylinder length=0.005 radius=0.127; visual mesh filename=Falcon_PropellerCCW.dae scale=1.0 1.0 1.0
- link Falcon3/rotor_0: geometry collision cylinder length=0.005 radius=0.127; visual mesh filename=Falcon_PropellerCW.dae scale=1.0 1.0 1.0
- link Falcon3/rotor_3: geometry collision cylinder length=0.005 radius=0.127; visual mesh filename=Falcon_PropellerCCW.dae scale=1.0 1.0 1.0
Joints:
- joint Falcon1/base_joint: origin xyz=0 0 0.00 rpy=0 0 0 -> xyz=0 0 0.00 rpy=0 0 1.5708
- joint Falcon1/rotor_0_joint: origin xyz=0.075 -0.075 0.05 rpy=0 0 0 -> xyz=0.075 0.075 0.02 rpy=0 0 0
- joint Falcon1/rotor_1_joint: origin xyz=-0.075 0.075 0.05 rpy=0 0 0 -> xyz=0.075 -0.075 0.02 rpy=0 0 0
- joint Falcon1/rotor_2_joint: origin xyz=-0.075 -0.075 0.05 rpy=0 0 0 -> xyz=-0.075 -0.075 0.02 rpy=0 0 0
- joint Falcon1/rotor_3_joint: origin xyz=0.075 0.075 0.05 rpy=0 0 0 -> xyz=-0.075 0.075 0.02 rpy=0 0 0
- joint Falcon2/base_joint: origin xyz=0 0 0.0 rpy=0 0 0 -> xyz=0 0 0.0 rpy=0 0 1.5708
- joint Falcon2/rotor_0_joint: origin xyz=0.075 -0.075 0.05 rpy=0 0 0 -> xyz=0.075 0.075 0.02 rpy=0 0 0
- joint Falcon2/rotor_1_joint: origin xyz=-0.075 0.075 0.05 rpy=0 0 0 -> xyz=0.075 -0.075 0.02 rpy=0 0 0
- joint Falcon2/rotor_2_joint: origin xyz=-0.075 -0.075 0.05 rpy=0 0 0 -> xyz=-0.075 -0.075 0.02 rpy=0 0 0
- joint Falcon2/rotor_3_joint: origin xyz=0.075 0.075 0.05 rpy=0 0 0 -> xyz=-0.075 0.075 0.02 rpy=0 0 0
- joint Falcon3/base_joint: origin xyz=0 0 0.0 rpy=0 0 0 -> xyz=0 0 0.0 rpy=0 0 1.5708
- joint Falcon3/rotor_0_joint: origin xyz=0.075 -0.075 0.05 rpy=0 0 0 -> xyz=0.075 0.075 0.02 rpy=0 0 0
- joint Falcon3/rotor_1_joint: origin xyz=-0.075 0.075 0.05 rpy=0 0 0 -> xyz=0.075 -0.075 0.02 rpy=0 0 0
- joint Falcon3/rotor_2_joint: origin xyz=-0.075 -0.075 0.05 rpy=0 0 0 -> xyz=-0.075 -0.075 0.02 rpy=0 0 0
- joint Falcon3/rotor_3_joint: origin xyz=0.075 0.075 0.05 rpy=0 0 0 -> xyz=-0.075 0.075 0.02 rpy=0 0 0

Commit message: realistic flycrane model

File: exts/MARL_mav_carry_ext/MARL_mav_carry_ext/assets/data/AMR/flycrane_data/flycrane.urdf (robot description, URDF)
Before this commit: robot flycrane, 95 links, 94 joints
Joints:
- joint Falcon1/base_joint: origin xyz=0 0 0.00 rpy=0 0 1.5708 -> xyz=0 0 0.03 rpy=0 0 1.5708
- joint Falcon1/rotor_0_joint: origin xyz=0.075 0.075 0.02 rpy=0 0 0 -> xyz=0.075 0.075 0.05 rpy=0 0 0
- joint Falcon1/rotor_1_joint: origin xyz=0.075 -0.075 0.02 rpy=0 0 0 -> xyz=0.075 -0.075 0.05 rpy=0 0 0
- joint Falcon1/rotor_2_joint: origin xyz=-0.075 -0.075 0.02 rpy=0 0 0 -> xyz=-0.075 -0.075 0.05 rpy=0 0 0
- joint Falcon1/rotor_3_joint: origin xyz=-0.075 0.075 0.02 rpy=0 0 0 -> xyz=-0.075 0.075 0.05 rpy=0 0 0
- joint Falcon2/base_joint: origin xyz=0 0 0.0 rpy=0 0 1.5708 -> xyz=0 0 0.03 rpy=0 0 1.5708
- joint Falcon2/rotor_0_joint: origin xyz=0.075 0.075 0.02 rpy=0 0 0 -> xyz=0.075 0.075 0.05 rpy=0 0 0
- joint Falcon2/rotor_1_joint: origin xyz=0.075 -0.075 0.02 rpy=0 0 0 -> xyz=0.075 -0.075 0.05 rpy=0 0 0
- joint Falcon2/rotor_2_joint: origin xyz=-0.075 -0.075 0.02 rpy=0 0 0 -> xyz=-0.075 -0.075 0.05 rpy=0 0 0
- joint Falcon2/rotor_3_joint: origin xyz=-0.075 0.075 0.02 rpy=0 0 0 -> xyz=-0.075 0.075 0.05 rpy=0 0 0
- joint Falcon3/base_joint: origin xyz=0 0 0.0 rpy=0 0 1.5708 -> xyz=0 0 0.03 rpy=0 0 1.5708
- joint Falcon3/rotor_0_joint: origin xyz=0.075 0.075 0.02 rpy=0 0 0 -> xyz=0.075 0.075 0.05 rpy=0 0 0
- joint Falcon3/rotor_1_joint: origin xyz=0.075 -0.075 0.02 rpy=0 0 0 -> xyz=0.075 -0.075 0.05 rpy=0 0 0
- joint Falcon3/rotor_2_joint: origin xyz=-0.075 -0.075 0.02 rpy=0 0 0 -> xyz=-0.075 -0.075 0.05 rpy=0 0 0
- joint Falcon3/rotor_3_joint: origin xyz=-0.075 0.075 0.02 rpy=0 0 0 -> xyz=-0.075 0.075 0.05 rpy=0 0 0
- joint rope_1_sphere_joint_0_joint_x: origin xyz=0.27 0.22 0.14 rpy=0 0 0 -> xyz=0.27 0.22 0.14 rpy=-1 0 0
- joint rope_2_sphere_joint_0_joint_x: origin xyz=0.27 -0.22 0.14 rpy=0 0 0 -> xyz=0.27 -0.22 0.14 rpy=1 0 0
- joint rope_3_sphere_joint_0_joint_x: origin xyz=-0.27 0.0 0.14 rpy=0 0 0 -> xyz=-0.27 0.0 0.14 rpy=0 -1 0
