Commit message: flycrane model with offset

File: exts/MARL_mav_carry_ext/MARL_mav_carry_ext/assets/data/AMR/flycrane_rod_data/flycrane.urdf (robot description, URDF)
Before this commit: robot flycrane, 41 links, 40 joints
Joints:
- joint Falcon1/base_joint: origin xyz=0 0 0.03 rpy=0 0 1.5708 -> xyz=0 0 0.03 rpy=0 0 0
- joint Falcon2/base_joint: origin xyz=0 0 0.03 rpy=0 0 1.5708 -> xyz=0 0 0.03 rpy=0 0 0
- joint Falcon3/base_joint: origin xyz=0 0 0.03 rpy=0 0 1.5708 -> xyz=0 0 0.03 rpy=0 0 0
