Commit message: new mesh, temporary LLC, terminations and reward ideas

File: exts/MARL_mav_carry_ext/MARL_mav_carry_ext/assets/data/AMR/falcon_data/falcon.urdf (robot description, URDF)
Before this commit: robot Falcon, 6 links, 5 joints
Links:
- link Falcon/base_link_inertia: geometry collision box size=0.1 0.1 0.05; visual mesh filename=falcon_without_rotors.dae scale=1.0 1.0 1.0
- link Falcon/rotor_0: geometry collision cylinder length=0.005 radius=0.127; visual mesh filename=Falcon_PropellerCCW.dae scale=1.0 1.0 1.0
- link Falcon/rotor_1: geometry collision cylinder length=0.005 radius=0.127; visual mesh filename=Falcon_PropellerCCW.dae scale=1.0 1.0 1.0
- link Falcon/rotor_2: geometry collision cylinder length=0.005 radius=0.127; visual mesh filename=Falcon_PropellerCW.dae scale=1.0 1.0 1.0
- link Falcon/rotor_3: geometry collision cylinder length=0.005 radius=0.127; visual mesh filename=Falcon_PropellerCW.dae scale=1.0 1.0 1.0

File: exts/MARL_mav_carry_ext/MARL_mav_carry_ext/assets/data/AMR/flycrane_data/flycrane.urdf (robot description, URDF)
Before this commit: robot flycrane, 95 links, 94 joints
Links:
- link Falcon1/base_link_inertia: geometry collision box size=0.1 0.1 0.05; visual mesh filename=falcon_without_rotors.dae scale=1.0 1.0 1.0
- link Falcon1/rotor_0: geometry collision cylinder length=0.005 radius=0.127; visual mesh filename=Falcon_PropellerCCW.dae scale=1.0 1.0 1.0
- link Falcon1/rotor_1: geometry collision cylinder length=0.005 radius=0.127; visual mesh filename=Falcon_PropellerCCW.dae scale=1.0 1.0 1.0
- link Falcon1/rotor_2: geometry collision cylinder length=0.005 radius=0.127; visual mesh filename=Falcon_PropellerCW.dae scale=1.0 1.0 1.0
- link Falcon1/rotor_3: geometry collision cylinder length=0.005 radius=0.127; visual mesh filename=Falcon_PropellerCW.dae scale=1.0 1.0 1.0
- link Falcon2/base_link_inertia: geometry collision box size=0.1 0.1 0.05; visual mesh filename=falcon_without_rotors.dae scale=1.0 1.0 1.0
- link Falcon2/rotor_0: geometry collision cylinder length=0.005 radius=0.127; visual mesh filename=Falcon_PropellerCCW.dae scale=1.0 1.0 1.0
- link Falcon2/rotor_1: geometry collision cylinder length=0.005 radius=0.127; visual mesh filename=Falcon_PropellerCCW.dae scale=1.0 1.0 1.0
- link Falcon2/rotor_2: geometry collision cylinder length=0.005 radius=0.127; visual mesh filename=Falcon_PropellerCW.dae scale=1.0 1.0 1.0
- link Falcon2/rotor_3: geometry collision cylinder length=0.005 radius=0.127; visual mesh filename=Falcon_PropellerCW.dae scale=1.0 1.0 1.0
- link Falcon3/base_link_inertia: geometry collision box size=0.1 0.1 0.05; visual mesh filename=falcon_without_rotors.dae scale=1.0 1.0 1.0
- link Falcon3/rotor_0: geometry collision cylinder length=0.005 radius=0.127; visual mesh filename=Falcon_PropellerCCW.dae scale=1.0 1.0 1.0
- link Falcon3/rotor_1: geometry collision cylinder length=0.005 radius=0.127; visual mesh filename=Falcon_PropellerCCW.dae scale=1.0 1.0 1.0
- link Falcon3/rotor_2: geometry collision cylinder length=0.005 radius=0.127; visual mesh filename=Falcon_PropellerCW.dae scale=1.0 1.0 1.0
- link Falcon3/rotor_3: geometry collision cylinder length=0.005 radius=0.127; visual mesh filename=Falcon_PropellerCW.dae scale=1.0 1.0 1.0

Commit message: (direct) single falcon environment

File: exts/MARL_mav_carry_ext/MARL_mav_carry_ext/assets/data/AMR/falcon_data/falcon.urdf (robot description, URDF)
Before this commit: robot Falcon, 6 links, 5 joints
Links:
- link Falcon/rotor_0: geometry collision cylinder length=0.005 radius=0.127; visual mesh filename=Falcon_PropellerCW.dae scale=1.0 1.0 1.0
- link Falcon/rotor_3: geometry collision cylinder length=0.005 radius=0.127; visual mesh filename=Falcon_PropellerCCW.dae scale=1.0 1.0 1.0
Joints:
- joint Falcon/base_joint: origin xyz=0 0 0.03 rpy=0 0 0 -> xyz=0 0 0.0 rpy=0 0 1.5708
- joint Falcon/rotor_0_joint: origin xyz=0.075 -0.075 0.05 rpy=0 0 0 -> xyz=0.075 0.075 0.02 rpy=0 0 0
- joint Falcon/rotor_1_joint: origin xyz=-0.075 0.075 0.05 rpy=0 0 0 -> xyz=0.075 -0.075 0.02 rpy=0 0 0
- joint Falcon/rotor_2_joint: origin xyz=-0.075 -0.075 0.05 rpy=0 0 0 -> xyz=-0.075 -0.075 0.02 rpy=0 0 0
- joint Falcon/rotor_3_joint: origin xyz=0.075 0.075 0.05 rpy=0 0 0 -> xyz=-0.075 0.075 0.02 rpy=0 0 0

Commit message: update falcon model

File: exts/MARL_mav_carry_ext/MARL_mav_carry_ext/assets/data/AMR/falcon_data/falcon.urdf (robot description, URDF)
Before this commit: robot Falcon, 6 links, 5 joints
Joints:
- joint Falcon/base_joint: origin xyz=0 0 0.0 rpy=0 0 1.5708 -> xyz=0 0 0.03 rpy=0 0 0
- joint Falcon/rotor_0_joint: origin xyz=0.075 0.075 0.02 rpy=0 0 0 -> xyz=0.075 0.075 0.05 rpy=0 0 0
- joint Falcon/rotor_1_joint: origin xyz=0.075 -0.075 0.02 rpy=0 0 0 -> xyz=0.075 -0.075 0.05 rpy=0 0 0
- joint Falcon/rotor_2_joint: origin xyz=-0.075 -0.075 0.02 rpy=0 0 0 -> xyz=-0.075 -0.075 0.05 rpy=0 0 0
- joint Falcon/rotor_3_joint: origin xyz=-0.075 0.075 0.02 rpy=0 0 0 -> xyz=-0.075 0.075 0.05 rpy=0 0 0
